File: MPR121QR2_Keyboard.kicad_pcb (KiCad board)
At the start: 2 copper layers, 72 x 79 mm, 95 parts, among them J1 USB_C_Receptacle_USB2.0_16P, SW1 SW_Push, SW2 SW_Push, U1 AP1117-33, U2 W25Q128JVS, U3 LM358D, U4 RP2040, U5 MPR121QR2, Y1 Crystal_GND24

Commit message: rev0
Parts:
- added G***: LOGO, LOGO, F.Cu at (126.4, 49.8)
- added G***: LOGO, LOGO, B.Cu at (149.3, 89.7)
- added G***: LOGO, LOGO, F.Cu at (150.3, 52.5)
- added kibuzzard-680FD2EB: G***, kibuzzard-680FD2EB, F.Cu at (129.9, 61.2)
- moved swclk 1.67 mm to (116.5, 63.4)
- moved swdio 1.67 mm to (116.5, 60.4)
- renumbered TP3 to +5, TP4 to -, SW1 to boot, SW2 to rst, TP1 to swclk, TP2 to swdio
Routing:
- net +3.3V: track 0.00 -> 125.9 mm, vias 0 -> 5
- net RS: track 0.00 -> 70.5 mm, vias 0 -> 2
- net RES: track 0.00 -> 68.0 mm, vias 0 -> 2
- net MOSI: track 0.00 -> 61.2 mm, vias 0 -> 2
- net SCLK: track 0.00 -> 56.8 mm, vias 0 -> 2
- net IRQ: track 3.19 -> 57.7 mm, vias 0 -> 2
- net !SS: track 0.00 -> 54.3 mm, vias 0 -> 2
- net SDA_I2C: track 2.77 -> 51.6 mm, vias 0 -> 2
- net SCL_I2C: track 2.97 -> 50.1 mm, vias 0 -> 2
- net +3.3V_LDO: track 0.00 -> 41.1 mm
- net CURRENT_3V3: track 4.20 -> 41.5 mm, vias 0 -> 2
- net +5V USB: track 20.0 -> 46.7 mm
- net Earth: track 0.00 -> 26.0 mm, vias 0 -> 46
- net CURRENT_5V: track 20.4 -> 41.5 mm, vias 0 -> 2
- net Net-(U2-~{CS}): track 3.85 -> 24.9 mm, vias 0 -> 2
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- added copper zone on B.Cu, net Earth
- added copper zone on F.Cu, net Earth
Other:
- board text added: "by @madjogger"
